File: pcb/ACDetect.kicad_sch (KiCad schematic)
At the start: 8 parts, among them U1 ISO1211

Commit message: Manufactured board
Parts:
- C3: footprint Capacitor_SMD:C_0603_1608Metric -> Capacitor_SMD:C_0805_2012Metric; LCSC (none) -> C15850
- R2, R20: LCSC (none) -> C728174
Changed lines of the file:
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@@
       (effects (font (size 1.27 1.27)))
+    )
+    (property "LCSC" "C728174" (at 99.06 92.71 90)
+      (effects (font (size 1.27 1.27)) hide)
     )
     (pin "2")
@@
       (effects (font (size 1.27 1.27)) (justify left))
     )
-    (property "Footprint" "Capacitor_SMD:C_0603_1608Metric" (at 145.7452 93.98 0)
+    (property "Footprint" "Capacitor_SMD:C_0805_2012Metric" (at 145.7452 93.98 0)
       (effects (font (size 1.27 1.27)) hide)
     )
@@
     (property "Voltage" "15V" (at 149.86 93.98 0)
       (effects (font (size 1.27 1.27)))
+    )
+    (property "LCSC" "C15850" (at 144.78 90.17 0)
+      (effects (font (size 1.27 1.27)) hide)
     )
     (pin "2")
@@
       (effects (font (size 1.27 1.27)))
     )
+    (property "LCSC" "C728174" (at 99.06 72.39 90)
+      (effects (font (size 1.27 1.27)) hide)
+    )
     (pin "2")
