File: pcb/RS485.kicad_sch (KiCad schematic)
At the start: 5 parts, among them U8 THVD1400D

Commit message: Manufactured board
Parts:
- added R48: 120R, Resistor_SMD:R_1206_3216Metric, symbol Device:R
- R45, R46: LCSC (none) -> C22859
Connections:
- net RS485_A: now also R48.1
- net RS485_B: now also R48.2
Other:
- moved on the sheet: C24, D5
