File: pcb/RS485.kicad_sch (KiCad schematic)
At the start: 6 parts, among them U8 THVD1400D

Commit message: [0.2] Freeze for manufacture
Other:
- company: (none) -> Tilt Ltd / OpenEnergyMonitor
- title: (none) -> emonHP
Changed lines of the file:
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@@
 	(generator "eeschema")
 	(generator_version "9.0")
-	(paper "A4")
+	(paper "A2")
+	(title_block
+		(title "emonHP")
+		(date "2026-07-20")
+		(rev "0.2")
+		(company "Tilt Ltd / OpenEnergyMonitor")
+		(comment 1 "Creative Commons Attribution-ShareAlike 4.0 License")
+		(comment 2 "Commit: gitrev")
+	)
 	(junction
 		(at 102.87 90.17)
