File: pcb/emonHP.kicad_pcb (KiCad board)
At the start: 4 copper layers, 85 x 88 mm, 116 parts, among them CN1 CONN_03SCREW, CN3 Screw_Terminal_01x02, CN4 CONN_03SCREW, CN5 Screw_Terminal_01x02, J2 CONN_04PTH, J3 USB_C_Receptacle_USB2.0, J4 Conn_ARM_JTAG_SWD_10, J5 Conn_02x20_Odd_Even, Q1 Q_NPN_BEC_BRT, Q2 FDN5618P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

Commit message: Manufactured board
Parts:
- removed REF**: OSHW-Logo2_7.3x6mm_SilkScreen, Symbol:OSHW-Logo2_7.3x6mm_SilkScreen
- removed U10: SN74LVC1T45DRL, Package_TO_SOT_SMD:SOT-563
- added C16: 100n, Capacitor_SMD:C_0402_1005Metric, F.Cu at (112.5, 76.5)
- added J1: Conn_01x02, Connector_PinHeader_2.54mm:PinHeader_1x02_P2.54mm_Vertical, F.Cu at (110.3, 115.0)
- added R21: 10K, Resistor_SMD:R_0402_1005Metric, F.Cu at (124.0, 129.0)
- added R24: 10K, Resistor_SMD:R_0402_1005Metric, F.Cu at (121.0, 129.5)
- added R25: 10K, Resistor_SMD:R_0402_1005Metric, F.Cu at (122.5, 129.5)
- added R3: 10K, Resistor_SMD:R_0402_1005Metric, F.Cu at (124.0, 127.5)
- added R47: 5K1, Resistor_SMD:R_0402_1005Metric, F.Cu at (121.5, 112.0)
- added R48: 120R, Resistor_SMD:R_1206_3216Metric, F.Cu at (113.0, 126.5)
- C3: footprint Capacitor_SMD:C_0603_1608Metric -> Capacitor_SMD:C_0805_2012Metric
- Q1, Q3: value Q_NPN_BEC_BRT -> BC846
- R1: value 4K7 -> 5K1
- R29: value 47K -> 20K
- R30, R42: value 47K -> 10K
- R43: value 20K -> 10K
- moved D10 40.0 mm to (149.0, 138.5), turned to 45 degrees
- moved FD1 39.4 mm to (148.0, 101.5)
- moved R14 36.9 mm to (150.0, 139.5), turned to 45 degrees
- moved TP4 18.0 mm to (134.0, 106.0)
- moved TP3 16.1 mm to (134.0, 112.0)
- moved R45 2.92 mm to (116.5, 125.5), turned to 90 degrees
- moved R46 2.69 mm to (116.5, 122.0), turned to -90 degrees
- moved D5 2.06 mm to (113.5, 122.0), turned to 90 degrees
- moved R30 1.50 mm to (123.5, 112.0)
- moved C10 0.72 mm to (150.8, 136.7)
- moved R41 0.51 mm to (126.0, 112.0), turned to 0 degrees
- moved Q1 0.50 mm to (125.0, 115.0)
- moved Q2 0.50 mm to (121.5, 115.0)
- turned C20 to 0 degrees
- turned D8 to 0 degrees
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Connections:
- D10 pad 2: +3V3 -> /Vuc
- Q2 pad 1: Net-(Q1-C) -> Net-(Q2-G)
- Q2 pad 2: Net-(D8-A) -> /MBus/36V
- Q2 pad 3: /MBus/36V -> Net-(D8-A)
- R26 pad 1: +5V -> /MBUS_EN
- R26 pad 2: /MBUS_EN -> GND
- R30 pad 1: /MBus/36V -> Net-(Q2-G)
- U2 pad 37: unconnected-(U2-PB22-Pad37) -> /~{LED_ACT}
- U2 pad 9: /~{LED_ACT} -> /MBUS_OC
Routing:
- net /MBUS_OC: track 1.92 -> 96.3 mm, vias 0 -> 4
- net /~{LED_ACT}: track 32.4 -> 2.24 mm
- net /UART5_TX: track 49.3 -> 63.3 mm
- net +3V3: track 308.8 -> 295.2 mm, vias 9 -> 8
- net /MBus/36V: track 39.8 -> 49.9 mm, vias 3 -> 4
- net /RS485/RS485_B: track 7.39 -> 17.0 mm
- net /UART3_TX: track 72.2 -> 81.5 mm
- net +5V: track 171.5 -> 164.5 mm
- net /RS485/RS485_A: track 7.48 -> 13.3 mm
- net /UART3_RTS: track 47.0 -> 52.6 mm
- net Net-(Q2-G): track 0.00 -> 3.22 mm
- net /UART3_RX: track 50.3 -> 53.0 mm
- net Net-(U8-B): track 5.18 -> 2.48 mm
- net Net-(U8-A): track 5.18 -> 2.75 mm
- net Net-(Q3-B): track 11.9 -> 10.1 mm
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
Commit message: emonHP with Pi attachment
Parts:
- added D12: LED, LED_SMD:LED_0603_1608Metric, F.Cu at (143.0, 90.0)
- added R49: 470R, Resistor_SMD:R_0402_1005Metric, F.Cu at (143.0, 87.0)
- R13, R14, R8, R9: value 1K -> 470R
- U2: value ATSAMD21G15B-M -> ATSAMD21G16B-M
Routing:
- net Net-(D12-K): track 0.00 -> 1.70 mm
Other:
- board text added: "v0.2 (gitrev)"
- board text removed: "v0.1 (gitrev)"
