File: pcb/emonHP.kicad_pcb (KiCad board)
At the start: 4 copper layers, 85 x 88 mm, 124 parts, among them CN1 CONN_03SCREW, CN3 Screw_Terminal_01x02, CN4 CONN_03SCREW, CN5 Screw_Terminal_01x02, J1 Conn_01x02, J2 CONN_04PTH, J3 USB_C_Receptacle_USB2.0, J4 Conn_ARM_JTAG_SWD_10, J5 Conn_02x20_Odd_Even, Q1 BC846, Q2 FDN5618P, Q3 BC846, SW1 SW_Push, SW2 SW_Push, U1 ISO1211, U2 ATSAMD21G16B-M, U3 AP2112K-3.3, U4 RFM69CW, U5 LM2733XMF, U6 LM4040DBZ-5, U7 MC33072, U8 THVD1400D, U9 USBLC6-2P6

Commit message: [0.2] Freeze for manufacture
Parts:
- removed C12: 1u, Capacitor_SMD:C_0402_1005Metric
- removed C13: 2u2, Capacitor_SMD:C_0603_1608Metric
- removed CN3: Screw_Terminal_01x02, TerminalBlock_Phoenix:TerminalBlock_Phoenix_PT-1,5-2-3.5-H_1x02_P3.50mm_Horizontal
- removed D10: LED, LED_SMD:LED_0603_1608Metric
- removed J1: Conn_01x02, Connector_PinHeader_2.54mm:PinHeader_1x02_P2.54mm_Vertical
- added CN6: CONN_03SCREW, TerminalBlock_Phoenix:TerminalBlock_Phoenix_PT-1,5-3-3.5-H_1x03_P3.50mm_Horizontal, F.Cu at (108.0, 94.5)
- added CN7: CONN_03SCREW, TerminalBlock_Phoenix:TerminalBlock_Phoenix_PT-1,5-3-3.5-H_1x03_P3.50mm_Horizontal, F.Cu at (108.0, 107.5)
- added LED2: LED_Dual_KAK, ltst-s326:LTST-S326, F.Cu at (188.8, 71.0)
- added Q4: BC847, Package_TO_SOT_SMD:SOT-23, F.Cu at (182.0, 71.0)
- added Q5: BC847, Package_TO_SOT_SMD:SOT-23, F.Cu at (135.5, 97.0)
- added R50: 100K, Resistor_SMD:R_0402_1005Metric, F.Cu at (129.0, 99.5)
- added R51: 10R, Resistor_SMD:R_0603_1608Metric, F.Cu at (129.5, 98.0)
- added R52: 10K, Resistor_SMD:R_0402_1005Metric, F.Cu at (122.0, 95.5)
- added R53: 10K, Resistor_SMD:R_0402_1005Metric, F.Cu at (119.0, 100.0)
- added R54: 10K, Resistor_SMD:R_0402_1005Metric, F.Cu at (119.0, 101.0)
- added R55: 10K, Resistor_SMD:R_0402_1005Metric, F.Cu at (119.0, 102.0)
- added R56: 10K, Resistor_SMD:R_0402_1005Metric, F.Cu at (179.5, 71.0)
- added R57: 10K, Resistor_SMD:R_0402_1005Metric, F.Cu at (129.0, 100.5)
- added R58: 10K, Resistor_SMD:R_0402_1005Metric, F.Cu at (129.0, 101.5)
- added R59: 10K, Resistor_SMD:R_0402_1005Metric, F.Cu at (136.0, 99.5)
- C11: value 100n -> 2u2; footprint Capacitor_SMD:C_0402_1005Metric -> Capacitor_SMD:C_0603_1608Metric
- C14, C2, C7: footprint Capacitor_SMD:C_0603_1608Metric -> Capacitor_SMD:C_0402_1005Metric
- C3: value 10u -> 100n; footprint Capacitor_SMD:C_0805_2012Metric -> Capacitor_SMD:C_0402_1005Metric
- C9: value 100n -> 2u2
- CN5: value Screw_Terminal_01x02 -> CONN_03SCREW; footprint TerminalBlock_Phoenix:TerminalBlock_Phoenix_PT-1,5-2-5.0-H_1x02_P5.00mm_Horizontal -> TerminalBlock_Phoenix:TerminalBlock_Phoenix_PT-1,5-3-3.5-H_1x03_P3.50mm_Horizontal
- D11: value ABS6 -> ESD5Z3.3T5G; footprint Diode_SMD:Diode_Bridge_Diotec_ABS -> Diode_SMD:D_SOD-523
- D12: value LED -> ESD5Z3.3T5G; footprint LED_SMD:LED_0603_1608Metric -> Diode_SMD:D_SOD-523
- Q1, Q3: value BC846 -> BC847
- R15: value 1K -> 5K1
- R16: value 1K -> 470R
- R2: value 30K -> 5K1; footprint Resistor_SMD:R_2512_6332Metric -> Resistor_SMD:R_0402_1005Metric
- R20: value 30K -> 100K; footprint Resistor_SMD:R_2512_6332Metric -> Resistor_SMD:R_0402_1005Metric
- R22: value 15K -> 100K; footprint Resistor_SMD:R_0603_1608Metric -> Resistor_SMD:R_0402_1005Metric
- R23: value 560 -> 10K; footprint Resistor_SMD:R_0603_1608Metric -> Resistor_SMD:R_0402_1005Metric
- R31: footprint Resistor_SMD:R_0805_2012Metric -> Resistor_SMD:R_2512_6332Metric
- R44: value 1K -> 10K
- R49: value 470R -> 100K
- U1: value ISO1211 -> STM32C031K6Ux; footprint Package_SO:SOIC-8_3.9x4.9mm_P1.27mm -> Package_DFN_QFN:QFN-32-1EP_5x5mm_P0.5mm_EP3.45x3.45mm
- U2: value ATSAMD21G16B-M -> AP22814AW5; footprint Package_DFN_QFN:QFN-48-1EP_7x7mm_P0.5mm_EP5.15x5.15mm -> Package_TO_SOT_SMD:SOT-23-5
- U9: value USBLC6-2P6 -> LM393; footprint Package_TO_SOT_SMD:SOT-666 -> Package_SO:SOIC-8_3.9x4.9mm_P1.27mm
- moved FB2 77.1 mm to (179.0, 142.5), turned to -90 degrees
- moved R14 76.9 mm to (185.0, 71.0), turned to 0 degrees
- moved C14 75.8 mm to (178.5, 141.0)
- moved C15 75.5 mm to (178.0, 142.5), turned to 90 degrees
- moved R16 70.2 mm to (185.0, 70.0), turned to 0 degrees
- moved R20 69.9 mm to (185.0, 72.0)
- moved SMA1 68.0 mm to (185.5, 141.0)
- moved R17 66.8 mm to (178.0, 133.5), turned to -90 degrees
- moved R12 65.5 mm to (186.0, 132.5), turned to 0 degrees
- moved C4 64.6 mm to (186.5, 131.0), turned to 180 degrees
- moved D1 64.6 mm to (186.0, 134.0)
- moved SW2 63.8 mm to (174.0, 78.5), turned to 180 degrees
- moved U4 62.1 mm to (168.5, 139.0), turned to 180 degrees
- moved C7 62.0 mm to (163.6, 81.6), turned to 0 degrees
- moved U3 61.9 mm to (186.5, 128.0), turned to 90 degrees
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Connections:
- net /MBus/DIFF_5V renamed /MBus/V_{sense}x5
- C10 pad 1: /Vuc -> +3V3
- C11 pad 1: /Vuc -> GND
- C11 pad 2: GND -> Net-(U9B--)
- C3 pad 1: Net-(D11-+) -> +3V3
- C3 pad 2: GND1 -> GND
- C8 pad 1: /Vuc -> Net-(U1-VDD)
- C9 pad 1: /Vuc -> /5V_{RPi}
- CN5 pad 1: /ACDetect/AC0 -> GND
- CN5 pad 2: /ACDetect/AC1 -> /OPA2
- D11 pad 1: Net-(D11-+) -> /OPA2
- D11 pad 2: GND1 -> GND
- D12 pad 1: Net-(D12-K) -> /OPA3
- D12 pad 2: /DHW_SENSE -> GND
- FB1 pad 2: /Vuc -> Net-(U1-VDD)
- J3 pad A6: /USB_D+ -> unconnected-(J3-D+-PadA6)
- J3 pad A7: /USB_D- -> unconnected-(J3-D--PadA7)
- J3 pad B6: /USB_D+ -> unconnected-(J3-D+-PadB6)
- J3 pad B7: /USB_D- -> unconnected-(J3-D--PadB7)
- J5 pad 12: unconnected-(J5-Pin_12-Pad12) -> /INTERRUPT
- J5 pad 15: /DHW_SENSE -> /OPA2
- J5 pad 18: /~{PI_PRESENT} -> /~{RESET}
- J5 pad 2: +5V -> /5V_{RPi}
- J5 pad 27: unconnected-(J5-Pin_27-Pad27) -> /OPA3
- J5 pad 36: unconnected-(J5-Pin_36-Pad36) -> /SWDIO
- J5 pad 38: unconnected-(J5-Pin_38-Pad38) -> /SWCLK
- J5 pad 4: +5V -> /5V_{RPi}
- Q1 pad 1: /UART5_TX -> Net-(Q1-B)
- R1 pad 2: +3V3 -> /OPA1_PU
- R11 pad 1: /Vuc -> +3V3
- R14 pad 1: Net-(D10-K) -> /~{LED_FW}
- R14 pad 2: /~{LED_ACT} -> Net-(LED2-K2)
- R15 pad 1: /UART3_TX_uc -> /OPA3
- R15 pad 2: /UART3_TX -> /OPA3_PU
- R16 pad 1: /UART3_RTS_uc -> /~{LED_POWER}
- R16 pad 2: /UART3_RTS -> Net-(LED2-K1)
- R2 pad 1: /ACDetect/AC1 -> /OPA2
- R2 pad 2: Net-(D11-Pad4) -> /OPA2_PU
- R20 pad 1: /ACDetect/AC0 -> /~{LED_FW}
- R20 pad 2: Net-(D11-Pad3) -> +3V3
- R22 pad 1: Net-(D11-+) -> /MBus/V_{sat}
- R22 pad 2: GND1 -> Net-(Q3-B)
- R23 pad 1: Net-(D11-+) -> /UART5_TX
- R23 pad 2: Net-(U1-IN) -> Net-(Q1-B)
- R41 pad 2: Net-(Q3-B) -> /MBus/V_{sat}
- R43 pad 2: /MBUS_OC -> Net-(U9A--)
- R44 pad 1: /MBUS_OC -> Net-(U9A--)
- R49 pad 1: Net-(D12-K) -> /RPI_PWR_EN
- R8 pad 1: /~{LED_STATUS} -> /~{LED_MBUS_EN}
- R9 pad 1: /~{LED_PROG} -> /~{LED_MBUS_ERR}
- U1 pad 1: +3V3 -> unconnected-(U1-PB9-Pad1)
- U1 pad 2: unconnected-(U1-EN-Pad2) -> GND
- U1 pad 3: /DHW_SENSE -> GND
- U1 pad 4: GND -> Net-(U1-VDD)
- U1 pad 5: unconnected-(U1-SUB-Pad5) -> GND
- U1 pad 6: GND1 -> /~{RESET}
- U1 pad 7: Net-(U1-IN) -> unconnected-(U1-PA0-Pad7)
- U1 pad 8: Net-(D11-+) -> unconnected-(U1-PA1-Pad8)
- U2 pad 1: unconnected-(U2-PA00-Pad1) -> /5V_{RPi}
- U2 pad 2: unconnected-(U2-PA01-Pad2) -> GND
- U2 pad 4: unconnected-(U2-PA03-Pad4) -> /RPI_PWR_EN
- U2 pad 5: GND -> +5V
- U7 pad 7: Net-(Q3-B) -> /MBus/V_{sat}
- U9 pad 1: /USB_D- -> /MBUS_OC
- U9 pad 2: GND -> Net-(U9A--)
- U9 pad 3: /USB_D+ -> Net-(U9A-+)
- U9 pad 4: /USB_D+ -> GND
- U9 pad 5: +5V -> Net-(U9B-+)
- U9 pad 6: /USB_D- -> Net-(U9B--)
Routing:
- net +5V: track 164.5 -> 61.1 mm
- net /OPA2: track 0.00 -> 100.8 mm, vias 0 -> 2
- net /OPA3: track 0.00 -> 90.6 mm, vias 0 -> 2
- net /DHW_SENSE: track 73.6 -> 0.00 mm, vias 4 -> 0
- net /RFM_SEL: track 85.6 -> 18.4 mm, vias 3 -> 0
- net /RFM_MISO: track 80.1 -> 16.0 mm, vias 2 -> 0
- net /RPI_PWR_EN: track 0.00 -> 63.5 mm, vias 0 -> 2
- net /RFM_MOSI: track 80.7 -> 28.1 mm, vias 2 -> 0
- net /USB_D-: track 49.7 -> 0.00 mm, vias 2 -> 0
- net /USB_D+: track 49.2 -> 0.00 mm, vias 2 -> 0
- net /SWDIO: track 24.2 -> 73.3 mm, vias 0 -> 2
- net /RFM_SCK: track 81.2 -> 32.7 mm
- net +3V3: track 295.2 -> 343.4 mm, vias 8 -> 16
- net /SWCLK: track 30.6 -> 78.5 mm, vias 0 -> 2
- net /RFM_RESET: track 66.6 -> 21.8 mm, vias 4 -> 0
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- added copper zone on B.Cu, net +5V
- added copper zone on In2.Cu, net +5V
- added copper zone on F.Cu, net /5V_{RPi}
- removed copper zone on F.Cu, net +3V3
- removed copper zone on B.Cu, net GND1
Other:
- outline, holes or cut-outs redrawn
- board text added: "Angus Logan 2026"
- board text added: "MBus (+)"
- board text added: "MBus (-)"
- board text added: "RESET"
- board text added: "RS485 (A)"
- board text added: "RS485 (B)"
- board text added: "Signal (1)"
- board text added: "Signal (2)"
- board text added: "Signal (3)"
- board text added: "github.com/openenergymonitor/emonHP"
- board text added: "n/c"
- board text removed: "1: RESET 2: BOOT"
- board text removed: "5V"
- board text removed: "Angus Logan 2025"
- board text removed: "github.com/awjlogan/emonHP"
