File: pcb/emonHP.kicad_sch (KiCad schematic)
At the start: 73 parts, among them CN1 CONN_03SCREW, CN3 Screw_Terminal_01x02, CN4 CONN_03SCREW, CN5 Screw_Terminal_01x02, J1 Conn_01x02, J2 CONN_04PTH, J3 USB_C_Receptacle_USB2.0, J4 Conn_ARM_JTAG_SWD_10, J5 Conn_02x20_Odd_Even, SW1 SW_Push, SW2 SW_Push, U2 ATSAMD21G16B-M, U3 AP2112K-3.3, U4 RFM69CW, U9 USBLC6-2P6

Commit message: [0.2] Freeze for manufacture
Parts:
- removed C10, C11: 100n, Capacitor_SMD:C_0402_1005Metric, symbol Device:C
- removed C12: 1u, Capacitor_SMD:C_0402_1005Metric, symbol Device:C
- removed C13: 2u2, Capacitor_SMD:C_0603_1608Metric, symbol Device:C
- removed CN3: Screw_Terminal_01x02, TerminalBlock_Phoenix:TerminalBlock_Phoenix_PT-1,5-2-3.5-H_1x02_P3.50mm_Horizontal, symbol Connector:Screw_Terminal_01x02
- removed CN5: Screw_Terminal_01x02, TerminalBlock_Phoenix:TerminalBlock_Phoenix_PT-1,5-2-5.0-H_1x02_P5.00mm_Horizontal, symbol Connector:Screw_Terminal_01x02
- removed D10, D12: LED, LED_SMD:LED_0603_1608Metric, symbol Device:LED
- removed J1: Conn_01x02, Connector_PinHeader_2.54mm:PinHeader_1x02_P2.54mm_Vertical, symbol Connector_Generic:Conn_01x02
- removed U2: ATSAMD21G16B-M, Package_DFN_QFN:QFN-48-1EP_7x7mm_P0.5mm_EP5.15x5.15mm, symbol MCU_Microchip_SAMD:ATSAMD21G16B-M
- removed U9: USBLC6-2P6, Package_TO_SOT_SMD:SOT-666, symbol Power_Protection:USBLC6-2P6
- added C1, C3: 100n, Capacitor_SMD:C_0402_1005Metric, symbol Device:C
- added CN5, CN6, CN7: CONN_03SCREW, TerminalBlock_Phoenix:TerminalBlock_Phoenix_PT-1,5-3-3.5-H_1x03_P3.50mm_Horizontal, symbol Connector:Screw_Terminal_01x03
- added D11, D12: ESD5Z3.3T5G, Diode_SMD:D_SOD-523, symbol Diode:ESD5Zxx
- added LED2: LED_Dual_KAK, ltst-s326:LTST-S326, symbol Device:LED_Dual_KAK
- added Q4: BC847, Package_TO_SOT_SMD:SOT-23, symbol Transistor_BJT:BC847
- added R2: 5K1, Resistor_SMD:R_0402_1005Metric, symbol Device:R
- added R20: 100K, Resistor_SMD:R_0402_1005Metric, symbol Device:R
- added R56: 10K, Resistor_SMD:R_0402_1005Metric, symbol Device:R
- added U1: STM32C031K6Ux, Package_DFN_QFN:QFN-32-1EP_5x5mm_P0.5mm_EP3.45x3.45mm, symbol MCU_ST_STM32C0:STM32C031K6Ux
- added U2: AP22814AW5, Package_TO_SOT_SMD:SOT-23-5, symbol Power_Management:AP22814AW5
- C14, C7: footprint Capacitor_SMD:C_0603_1608Metric -> Capacitor_SMD:C_0402_1005Metric; LCSC C23630 -> C12530
- C2: footprint Capacitor_SMD:C_0603_1608Metric -> Capacitor_SMD:C_0402_1005Metric; LCSC C23630 -> C12530; Voltage 16V -> (none)
- C9: value 100n -> 2u2; LCSC C1525 -> C12530; Voltage (none) -> 6V
- CN1, CN4: LCSC (none) -> C3582477
- J5: LCSC (none) -> C9900171940
- R15: value 1K -> 5K1; LCSC C11702 -> C25905
- R16: value 1K -> 470R; LCSC C11702 -> C25117
- R49: value 470R -> 100K; LCSC C25117 -> C25741
- SW1: now fitted
Connections:
- net UART3_TX_uc is gone; now on net OPA3: R15.1
- net ~{PI_PRESENT} is gone; now on net ~{RESET}: J5.18 (Pin_18)
- net +3V3: now also R11.1, C1.1, C3.1, CN5.3 (Pin_3), CN6.3 (Pin_3), LED2.2 (A), R20.2; no longer R1.2
- net +5V: now also U2.5 (IN); no longer J5.2 (Pin_2), J5.4 (Pin_4)
- net GND: now also C1.2, C3.2, CN5.1 (Pin_1), CN6.1 (Pin_1), CN7.3 (Pin_3), D11.2 (A), D12.2 (A), Q4.2 (E), U1.2 (PC14), U1.3 (PC15), U1.33 (VSS), U1.5 (VSS), U2.2 (GND)
- net I2C_SCL: now also U1.19 (PA9)
- net I2C_SDA: now also U1.21 (PA10)
- net MBUS_EN: now also U1.16 (PB1)
- net MBUS_OC: now also U1.15 (PB0)
- net MBus/MBUS_A: now also CN7.2 (Pin_2)
- net OPA1: now also U1.9 (PA2)
- net SWCLK: now also J5.38 (Pin_38), U1.25 (PA14)
- net SWDIO: now also J5.36 (Pin_36), U1.24 (PA13)
- net UART0_RX: now also U1.31 (PB7)
- net UART0_TX: now also U1.30 (PB6)
- net UART3_RTS: no longer R16.2
- net UART3_TX: no longer R15.2
- net ~{LCD_BUTTON}: now also U1.26 (PA15)
- net ~{RESET}: now also U1.6 (PF2)
- net RPI_PWR_EN: now reaches R49.1
- net RPI_PWR_EN: now also U1.32 (PB8), U2.4 (EN)
- net ~{LED_FW}: now reaches R14.1
- net ~{LED_FW}: now also R20.1, R56.1, U1.27 (PB3)
- net INTERRUPT: now reaches J5.12 (Pin_12)
- net INTERRUPT: now also U1.23 (PA12)
- net OPA3: now reaches J5.27 (Pin_27)
- net OPA3: now also CN6.2 (Pin_2), D12.1 (K), U1.13 (PA6)
- net DHW_SENSE renamed OPA2
- net OPA2: now also CN5.2 (Pin_2), D11.1 (K), R2.1, U1.11 (PA4)
- net UART3_RTS_uc renamed ~{LED_POWER}
- net ~{LED_POWER}: now also Q4.3 (C)
- net USB_D+: no longer names the net of J3.A6 (D+)
- net USB_D+: no longer J3.B6 (D+)
- net USB_D-: no longer names the net of J3.A7 (D-)
- net USB_D-: no longer J3.B7 (D-)
- net Vuc: no longer names the net of C8.1, FB1.2
- net Vuc: now also U1.4 (VDD); no longer C9.1, R11.1
- net ~{LED_ACT}: no longer names the net of R14.2
- net ~{LED_ACT}: now also LED2.3 (K2)
- net ~{LED_PROG} renamed ~{LED_MBUS_ERR}
- net ~{LED_MBUS_ERR}: now also U1.28 (PB4)
- net ~{LED_STATUS} renamed ~{LED_MBUS_EN}
- net ~{LED_MBUS_EN}: now also U1.29 (PB5)
- new net: Q4.1 (B), R56.2
- new net: LED2.1 (K1), R16.2
- new net 5V_{RPi}: C9.1, J5.2 (Pin_2), J5.4 (Pin_4), U2.1 (OUT)
- new net OPA1_PU: R1.2, U1.10 (PA3)
- new net OPA2_PU: R2.2, U1.12 (PA5)
- new net OPA3_PU: R15.2, U1.14 (PA7)
- no-connect marks 28 -> 27
Other:
- removed sheet ACDetect
- sheet MBus ports: added ~{MBUS_OC}; removed MBUS_OC
- note added: "K1 is RED."
- note removed: "SERCOM0"
- note removed: "SERCOM1"
- note removed: "SERCOM2"
- note removed: "SERCOM3"
- note removed: "SERCOM4"
- company: OpenEnergyMonitor / Tilt Ltd (Angus Logan) -> Tilt Ltd / OpenEnergyMonitor
- moved on the sheet: C16, C4, C5, C6, C7, C8, CN1, CN4, D2, D4, FB1, H3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
