File: pcb/mbus.kicad_sch (KiCad schematic)
At the start: 26 parts, among them Q1 BC846, Q2 FDN5618P, Q3 BC846, U6 LM4040DBZ-5, U7 MC33072

Commit message: [0.2] Freeze for manufacture
Parts:
- removed Q1, Q3: BC846, Package_TO_SOT_SMD:SOT-23, symbol Transistor_BJT:BC846
- added C10: 100n, Capacitor_SMD:C_0402_1005Metric, symbol Device:C
- added C11: 2u2, Capacitor_SMD:C_0603_1608Metric, symbol Device:C
- added Q1, Q3, Q5: BC847, Package_TO_SOT_SMD:SOT-23, symbol Transistor_BJT:BC847
- added R22, R50: 100K, Resistor_SMD:R_0402_1005Metric, symbol Device:R
- added R23, R52, R53, R54, R55, R57, R58, R59: 10K, Resistor_SMD:R_0402_1005Metric, symbol Device:R
- added R51: 10R, Resistor_SMD:R_0603_1608Metric, symbol Device:R
- added U9: LM393, Package_SO:SOIC-8_3.9x4.9mm_P1.27mm, symbol Comparator:LM393
- R31: footprint Resistor_SMD:R_0805_2012Metric -> Resistor_SMD:R_2512_6332Metric; LCSC C17408 -> C840600; MPN ERJ-P06J101V -> CRM2512-JW-101ELF; Manufacturer Panasonic -> Bourns; Mouser 667-ERJ-P06J101V -> 652-CRM2512-JW101ELF; Power 0.5W -> 2W
- R44: value 1K -> 10K; LCSC C11702 -> C25744
Connections:
- net +3V3: now also C10.1, R50.2, R52.2, R53.1, R57.1, U9.8 (V+)
- net GND: now also C10.2, C11.1, Q1.2 (E), Q3.2 (E), Q5.2 (E), R54.2, R58.2, U9.4 (V-)
- net Rx: now also Q3.3 (C), R59.1
- net Tx: now also R23.1
- net at R30.2: now also Q1.3 (C)
- net V_{sat}: now reaches R41.2, U7.7
- net V_{sat}: now also R22.1
- net DIFF_5V renamed V_{sense}x5
- net MBUS_OC: no longer names the net of R43.2, R44.1
- net MBUS_OC: now also U9.2 (-)
- new net: Q1.1 (B), R23.2
- new net: C11.2, R50.1, R51.2, U9.6 (-)
- new net: R53.2, R54.1, R55.1, U9.3 (+)
- new net: R57.2, R58.1, U9.5 (+)
- new net: Q5.1 (B), R59.2
- new net: Q5.3 (C), R51.1
- new net: Q3.1 (B), R22.2
- new net ~{MBUS_OC}: R52.1, R55.2, U9.1, U9.7
Other:
- note added: "(V > 5) saturates at Vss"
- note removed: "(V > 5) saturates at 0V"
- moved on the sheet: C22, C23, D8, D9, Q2, R29, R30, R31, R32, R33, R34, R35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
